Commit message: Update court.urdf

File: court.urdf (robot description, URDF)
Before this commit: robot basketball_court, 1 links, 0 joints
Links:
- link court: geometry visual box size=0.023928 0.012700 0.010000; visual box size=0.023928 0.012700 0.010000

Commit message: Update rim hopefully

File: court.urdf (robot description, URDF)
Before this commit: robot basketball_court, 1 links, 0 joints
Links:
- link court: geometry visual box size=0.024759 0.015875 0.015875; visual box size=0.024759 0.015875 0.015875
